Commit message: catkin_make success & adaptation for running impact_sim

File: impactor/impact_sim/config/model/quadrotor.urdf (robot description, URDF)
Before this commit: robot quadrotor, 1 links, 0 joints
Links:
- link base_link: geometry collision box size=.36 .4 .06; visual mesh filename=/home/stark/impactor_ws/src/IMPACTOR/impactor/impact_sim/co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 scale=0.001
